File: hardware/jarvis-2.0.brd (EAGLE design)
At the start: 73.6 x 67.3 mm, 35 parts, among them IC1 ATMEGA8L, IC2 WT588D, IC3 HC-05, T1 2N3904, T2 2N3904, T3 2N3904, T4 2N3904, T5 2N3904

Commit message: Fixed value of eyes leds resitor.
Parts:
- R8: value 180 -> 68
Changed lines of the file:
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@@
 <element name="C4" library="capacitor-wima" package="C2.5-2" value="100nF" x="24.765" y="24.13" rot="R90"/>
 <element name="C5" library="rcl" package="E5-5" value="100uF" x="23.495" y="54.61" rot="R270"/>
-<element name="R8" library="resistor" package="0204/7" value="180" x="24.765" y="8.89" rot="R90"/>
+<element name="R8" library="resistor" package="0204/7" value="68" x="24.765" y="8.89" rot="R90"/>
 <element name="R9" library="resistor" package="0204/7" value="" x="13.97" y="57.785"/>
 <element name="R10" library="resistor" package="0204/7" value="" x="56.515" y="42.545" rot="R270"/>
