File: hardware/jarvis-2.0.sch (EAGLE design)
At the start: 35 parts, among them IC1 ATMEGA8L, IC2 WT588D, IC3 HC-05, T1 2N3904, T2 2N3904, T3 2N3904, T4 2N3904, T5 2N3904

Commit message: Fixed value of eyes leds resitor.
Parts:
- R8: value 180 -> 68
Changed lines of the file:
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@@
 <part name="C5" library="rcl" deviceset="CPOL-EU" device="E5-5" value="100uF"/>
 <part name="GND15" library="supply1" deviceset="GND" device=""/>
-<part name="R8" library="resistor" deviceset="R-EU_" device="0204/7" value="180"/>
+<part name="R8" library="resistor" deviceset="R-EU_" device="0204/7" value="68"/>
 <part name="R9" library="resistor" deviceset="R-EU_" device="0204/7"/>
 <part name="R10" library="resistor" deviceset="R-EU_" device="0204/7"/>
